File: PCBs/mdac-attenuator/mdac-attenuator.sch (KiCad schematic (older format))
At the start: 34 parts, among them J1 Conn_01x06_Male, J2 Conn_01x06_Male, U1 AD8599, U2 DAC8812ICPWG4

Commit message: Updated the mdac-attenuator to work with kicad 5.
Changed lines of the file:
@@
 EESchema Schematic File Version 4
-LIBS:mdac-attenuator-cache
-EELAYER 26 0
+EELAYER 30 0
 EELAYER END
 $Descr A4 11693 8268
@@
 $EndComp
 $Comp
-L power:VDD #PWR0109
-U 1 1 5C5BB6C7
-P 2800 950
-F 0 "#PWR0109" H 2800 800 50  0001 C CNN
-F 1 "VDD" H 2817 1123 50  0000 C CNN
-F 2 "" H 2800 950 50  0001 C CNN
-F 3 "" H 2800 950 50  0001 C CNN
-	1    2800 950
-	1    0    0    -1
-$EndComp
-$Comp
 L Device:LED LED1
 U 1 1 5C5CA887
@@
 Connection ~ 2200 1850
 Wire Wire Line
-	2200 1850 2800 1850
+	2200 1850 2500 1850
 Wire Wire Line
 	2200 1300 2200 1000
 Connection ~ 2200 1000
-Wire Wire Line
-	2200 1000 2800 1000
 $Comp
 L power:GNDD #PWR0110
@@
 	1    0    0    -1
 $EndComp
+$Comp
+L power:PWR_FLAG #FLG0101
+U 1 1 612C57C3
+P 2450 800
+F 0 "#FLG0101" H 2450 875 50  0001 C CNN
+F 1 "PWR_FLAG" H 2450 973 50  0000 C CNN
+F 2 "" H 2450 800 50  0001 C CNN
+F 3 "~" H 2450 800 50  0001 C CNN
+	1    2450 800
+	1    0    0    -1
+$EndComp
+$Comp
+L power:VDD #PWR0109
+U 1 1 5C5BB6C7
+P 2800 950
+F 0 "#PWR0109" H 2800 800 50  0001 C CNN
+F 1 "VDD" H 2817 1123 50  0000 C CNN
+F 2 "" H 2800 950 50  0001 C CNN
+F 3 "" H 2800 950 50  0001 C CNN
+	1    2800 950
+	1    0    0    -1
+$EndComp
+$Comp
+L power:PWR_FLAG #FLG0102
+U 1 1 612ED7CB
+P 2500 2150
+F 0 "#FLG0102" H 2500 2225 50  0001 C CNN
+F 1 "PWR_FLAG" H 2500 2323 50  0000 C CNN
+F 2 "" H 2500 2150 50  0001 C CNN
+F 3 "~" H 2500 2150 50  0001 C CNN
+	1    2500 2150
+	1    0    0    1
+$EndComp
+$Comp
+L power:PWR_FLAG #FLG0103
+U 1 1 61305D76
+P 5150 800
+F 0 "#FLG0103" H 5150 875 50  0001 C CNN
+F 1 "PWR_FLAG" H 5150 973 50  0000 C CNN
+F 2 "" H 5150 800 50  0001 C CNN
+F 3 "~" H 5150 800 50  0001 C CNN
+	1    5150 800
+	1    0    0    -1
+$EndComp
+Wire Wire Line
+	5150 800  5150 1050
+$Comp
+L power:PWR_FLAG #FLG0104
+U 1 1 6130D939
+P 5150 2150
+F 0 "#FLG0104" H 5150 2225 50  0001 C CNN
+F 1 "PWR_FLAG" H 5150 2323 50  0000 C CNN
+F 2 "" H 5150 2150 50  0001 C CNN
+F 3 "~" H 5150 2150 50  0001 C CNN
+	1    5150 2150
+	1    0    0    1
+$EndComp
+Wire Wire Line
+	5150 2150 5150 1850
+Wire Wire Line
+	2200 1000 2450 1000
+Wire Wire Line
+	2450 800  2450 1000
+Connection ~ 2450 1000
+Wire Wire Line
+	2450 1000 2800 1000
+Wire Wire Line
+	2500 2150 2500 1850
+Connection ~ 2500 1850
+Wire Wire Line
+	2500 1850 2800 1850
 $EndSCHEMATC
